Commit message: 微调urdf

File: source/Dog/Dog/assets/RC/rc_dog/urdf/rcdog.urdf (robot description, URDF)
Before this commit: robot bbb, 17 links, 16 joints
Links:
- link base_link: geometry collision mesh filename=../meshes/base_link.STL; visual mesh filename=../meshes/base_link.STL
- link lb_calf_link: mass 0.0885710163289355 -> 0.0886411363789507; geometry collision mesh filename=../meshes/lb_calf_link.STL; visual mesh filename=../meshes/lb_calf_link.STL
- link lb_foot_link: geometry collision mesh filename=../meshes/lb_foot_link.STL; visual mesh filename=../meshes/lb_foot_link.STL
- link lb_hip_link: geometry collision mesh filename=../meshes/lb_hip_link.STL; visual mesh filename=../meshes/lb_hip_link.STL
- link lb_thigh_link: mass 0.658206324923643 -> 0.658933850403685; geometry collision mesh filename=../meshes/lb_thigh_link.STL; visual mesh filename=../meshes/lb_thigh_link.STL
- link lf_calf_link: mass 0.0885710163289359 -> 0.0886411364041483; geometry collision mesh filename=../meshes/lf_calf_link.STL; visual mesh filename=../meshes/lf_calf_link.STL
- link lf_foot_link: geometry collision mesh filename=../meshes/lf_foot_link.STL; visual mesh filename=../meshes/lf_foot_link.STL
- link lf_hip_link: geometry collision mesh filename=../meshes/lf_hip_link.STL; visual mesh filename=../meshes/lf_hip_link.STL
- link lf_thigh_link: mass 0.658206351594895 -> 0.658934018099903; geometry collision mesh filename=../meshes/lf_thigh_link.STL; visual mesh filename=../meshes/lf_thigh_link.STL
- link rb_calf_link: mass 0.0887112564289659 -> 0.0886411363789507; geometry collision mesh filename=../meshes/rb_calf_link.STL; visual mesh filename=../meshes/rb_calf_link.STL
- link rb_foot_link: geometry collision mesh filename=../meshes/rb_foot_link.STL; visual mesh filename=../meshes/rb_foot_link.STL
- link rb_hip_link: geometry collision mesh filename=../meshes/rb_hip_link.STL; visual mesh filename=../meshes/rb_hip_link.STL
- link rb_thigh_link: mass 0.659661375883727 -> 0.658933850403685; geometry collision mesh filename=../meshes/rb_thigh_link.STL; visual mesh filename=../meshes/rb_thigh_link.STL
- link rf_calf_link: mass 0.0887112564793606 -> 0.0886411364041483; geometry collision mesh filename=../meshes/rf_calf_link.STL; visual mesh filename=../meshes/rf_calf_link.STL
- link rf_foot_link: geometry collision mesh filename=../meshes/rf_foot_link.STL; visual mesh filename=../meshes/rf_foot_link.STL
- link rf_hip_link: geometry collision mesh filename=../meshes/rf_hip_link.STL; visual mesh filename=../meshes/rf_hip_link.STL
- link rf_thigh_link: mass 0.659661684604912 -> 0.658934018099903; geometry collision mesh filename=../meshes/rf_thigh_link.STL; visual mesh filename=../meshes/rf_thigh_link.STL
Joints:
- joint lb_hip_roll_joint: axis -1 0 0 -> 1 0 0
- joint lb_knee_joint: axis 0 -1 0 -> 0 1 0
- joint lf_hip_pitch_joint: axis 0 -1 0 -> 0 1 0
- joint lf_hip_roll_joint: axis -1 0 0 -> 1 0 0
- joint lf_knee_joint: axis 0 -1 0 -> 0 1 0
- joint rb_hip_pitch_joint: axis 0 -1 0 -> 0 1 0
- joint rb_hip_roll_joint: axis -1 0 0 -> 1 0 0
- joint rb_knee_joint: axis 0 -1 0 -> 0 1 0
- joint rf_hip_pitch_joint: axis 0 -0.999962861141045 -0.00861837215575348 -> 0 1 0
- joint rf_knee_joint: axis 0 0.999962861141045 0.00861837215574936 -> 0 1 0
